Commit message: final ros2 humble

File: urdf/_d435.urdf.xacro (robot description, xacro)
@@ -45,5 +45,5 @@
     <link name="${name}_link">
       <visual>
-      <origin xyz="${d435_cam_mount_from_center_offset} ${-d435_cam_depth_py} 0" rpy="${M_PI/2} 0 ${M_PI/2}"/>
+      <origin xyz="${d435_cam_mount_from_center_offset} ${-d435_cam_depth_py} 0" rpy="0 0 0"/>
         <geometry>
           <!-- <box size="${d435_cam_width} ${d435_cam_height} ${d435_cam_depth}"/> -->

File: urdf/test_d435_camera.urdf.xacro (robot description, xacro)
@@ -4,5 +4,5 @@
   <link name="base_link" />
   <xacro:sensor_d435 name="camera" topics_ns="camera" parent="base_link" publish_pointcloud="true">
-    <origin xyz="0 0 0" rpy="0 0 0" />
+    <origin xyz="0 0 0" rpy="-1.57 0 -1.57" />
   </xacro:sensor_d435>
 </robot>

Commit message: phase 1

File: urdf/_d435.urdf.xacro (robot description, xacro)
@@ -45,5 +45,5 @@
     <link name="${name}_link">
       <visual>
-      <origin xyz="${d435_cam_mount_from_center_offset} ${-d435_cam_depth_py} 0" rpy="0 0 0"/>
+      <origin xyz="${d435_cam_mount_from_center_offset} ${-d435_cam_depth_py} 0" rpy="${-M_PI/2} 0 ${-M_PI/2}"/>
         <geometry>
           <!-- <box size="${d435_cam_width} ${d435_cam_height} ${d435_cam_depth}"/> -->

File: urdf/test_d435_camera.urdf.xacro (robot description, xacro)
@@ -3,6 +3,15 @@
   <xacro:include filename="$(find realsense2_description)/urdf/_d435.urdf.xacro" />
   <link name="base_link" />
+  <!-- <link name="camera_rotation_link"/>
+  <joint name="camera_rotation_joint" type="fixed">
+      <origin xyz="0 0 0" rpy="0 0 1.57" />
+      <parent link="base_link" />
+      <child link="camera_rotation_link" />
+  </joint> -->
   <xacro:sensor_d435 name="camera" topics_ns="camera" parent="base_link" publish_pointcloud="true">
-    <origin xyz="0 0 0" rpy="-1.57 0 -1.57" />
+    <!-- horizontal camera-->
+    <origin xyz="0 0 0" rpy="1.57 0 0" />
+    <!-- vertical camera-->
+    <!-- <origin xyz="0 0 0" rpy="0 1.57 0" />       -->
   </xacro:sensor_d435>
 </robot>

File: urdf/test_d435_multiple_cameras.urdf.xacro (robot description, xacro)
@@ -3,9 +3,9 @@
   <xacro:include filename="$(find realsense2_description)/urdf/_d435.urdf.xacro" />
   <link name="base_link" />
-  <sensor_d435 parent="base_link" name="camera1">
-    <origin xyz="0.1 0 0" rpy="0 0 0"/>
+  <sensor_d435 parent="base_link" name="camera_left" publish_pointcloud="true">
+    <origin xyz="0 -3 0" rpy="-1.57 0 -1.57"/>
   </sensor_d435>
-  <sensor_d435 parent="base_link" name="camera2">
-    <origin xyz="-0.1 0 0" rpy="0 0 3.1456"/>
+  <sensor_d435 parent="base_link" name="camera_right" publish_pointcloud="true">
+    <origin xyz="0 3 0" rpy="-1.57 0 -1.57"/>
   </sensor_d435>
 </robot>

Commit message: multiple camera 42deg

File: urdf/_d435.urdf.xacro (robot description, xacro)
@@ -45,5 +45,5 @@
     <link name="${name}_link">
       <visual>
-      <origin xyz="${d435_cam_mount_from_center_offset} ${-d435_cam_depth_py} 0" rpy="${-M_PI/2} 0 ${-M_PI/2}"/>
+      <origin xyz="${d435_cam_mount_from_center_offset} ${-d435_cam_depth_py} 0" rpy="0 0 0"/>
         <geometry>
           <!-- <box size="${d435_cam_width} ${d435_cam_height} ${d435_cam_depth}"/> -->

File: urdf/test_d435_multiple_cameras.urdf.xacro (robot description, xacro)
@@ -3,9 +3,9 @@
   <xacro:include filename="$(find realsense2_description)/urdf/_d435.urdf.xacro" />
   <link name="base_link" />
-  <sensor_d435 parent="base_link" name="camera_left" publish_pointcloud="true">
-    <origin xyz="0 -3 0" rpy="-1.57 0 -1.57"/>
-  </sensor_d435>
-  <sensor_d435 parent="base_link" name="camera_right" publish_pointcloud="true">
-    <origin xyz="0 3 0" rpy="-1.57 0 -1.57"/>
-  </sensor_d435>
+  <xacro:sensor_d435 parent="base_link" name="camera_left" publish_pointcloud="true">
+    <origin xyz="0 0.3 0" rpy="-1.57 0 -2.3038"/>
+  </xacro:sensor_d435>
+  <xacro:sensor_d435 parent="base_link" name="camera_right" publish_pointcloud="true">
+    <origin xyz="0 -0.3 0" rpy="-1.57 0 -0.8378"/>
+  </xacro:sensor_d435>
 </robot>
